Commit message: first commit

File: hector_quadrotor/hector_quadrotor_description/urdf/quadrotor_hokuyo_utm30lx.urdf.xacro (robot description, xacro)
@@ -13,6 +13,6 @@
     <!-- Forward facing camera -->
     <xacro:include filename="$(find hector_sensors_description)/urdf/generic_camera.urdf.xacro" />
-    <xacro:generic_camera name="front_cam" parent="base_link" ros_topic="camera/image" cam_info_topic="camera/camera_info" update_rate="20" res_x="320" res_y="240" image_format="R8G8B8" hfov="90">
-      <origin xyz="0 0.0 -0.15" rpy="0 1.57 0"/>
+    <xacro:generic_camera name="front_cam" parent="base_link" ros_topic="camera/image" cam_info_topic="camera/camera_info" update_rate="10" res_x="320" res_y="240" image_format="R8G8B8" hfov="90">
+      <origin xyz="0.05 0.0 -0.06" rpy="0 0 0"/>
     </xacro:generic_camera>
 </robot>

Commit message: added hector_gazebo package to easily add more worlds or plugins and avoid ros path problems.

File: hector_quadrotor/hector_quadrotor_description/urdf/quadrotor_hokuyo_utm30lx.urdf.xacro (robot description, xacro)
@@ -14,5 +14,5 @@
     <xacro:include filename="$(find hector_sensors_description)/urdf/generic_camera.urdf.xacro" />
     <xacro:generic_camera name="front_cam" parent="base_link" ros_topic="camera/image" cam_info_topic="camera/camera_info" update_rate="10" res_x="320" res_y="240" image_format="R8G8B8" hfov="90">
-      <origin xyz="0.05 0.0 -0.06" rpy="0 0 0"/>
+      <origin xyz="0.0 0.0 -0.2" rpy="0 1.57 0"/>
     </xacro:generic_camera>
 </robot>
